File: Schematic and Layout/Rx.brd (EAGLE design)
At the start: 48.3 x 80 mm, 19 parts

Commit message: Add files via upload
Parts:
- U$10: value RES -> 100
- U$11, U$4: value RES -> 10K
- U$13: value LED_1206 -> LED_12V
- U$14: value CAP -> 470uF
- U$15: value RES -> 330
- U$16, U$6: value RES -> 1K
- U$18: value POWER_CONN -> 5V-12V
- U$20: value DIODE_Z_1005 -> 15V_Z
- U$5, U$7: value RES -> 100K
- moved U$11 1.91 mm to (40.6, 51.6)
Routing:
- net N$2: track 26.6 -> 24.4 mm
- net N$7: track 64.6 -> 62.7 mm
Other:
- board size 48.3 x 80 mm -> 44.5 x 80 mm
- board text added: "12V_VIN"
- board text removed: "VIN"
Changed lines of the file:
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@@
 <board>
 <plain>
-<wire x1="0" y1="0" x2="48.26" y2="0" width="0" layer="20"/>
-<wire x1="48.26" y1="0" x2="48.26" y2="80.01" width="0" layer="20"/>
-<wire x1="48.26" y1="80.01" x2="0" y2="80.01" width="0" layer="20"/>
+<wire x1="0" y1="0" x2="44.45" y2="0" width="0" layer="20"/>
+<wire x1="44.45" y1="0" x2="44.45" y2="80.01" width="0" layer="20"/>
+<wire x1="44.45" y1="80.01" x2="0" y2="80.01" width="0" layer="20"/>
 <wire x1="0" y1="80.01" x2="0" y2="0" width="0" layer="20"/>
-<text x="0.6985" y="7.1755" size="1.778" layer="21" rot="R270">VIN</text>
+<text x="0.6985" y="12.573" size="1.778" layer="21" rot="R270">12V_VIN</text>
 <text x="3.7465" y="51.8795" size="1.778" layer="21">LOAD</text>
 </plain>
@@
 </autorouter>
 <elements>
-<element name="U$1" library="Gas_Sensor_Lib_v1" package="SOT23" value="NMOS" x="38.608" y="76.327" rot="R90"/>
-<element name="U$2" library="Gas_Sensor_Lib_v1" package="D-PAK_TO252AA" value="PMOS" x="29.718" y="60.198" rot="R270"/>
-<element name="U$3" library="Gas_Sensor_Lib_v1" package="DIDOE_1206" value="DIODE_1206" x="11.43" y="58.4835"/>
-<element name="U$4" library="Gas_Sensor_Lib_v1" package="R1206" value="RES" x="32.258" y="76.454" rot="R180"/>
-<element name="U$5" library="Gas_Sensor_Lib_v1" package="R1206" value="RES" x="26.162" y="76.454" rot="R180"/>
-<element name="U$6" library="Gas_Sensor_Lib_v1" package="R1206" value="RES" x="42.6085" y="61.214" rot="R90"/>
-<element name="U$7" library="Gas_Sensor_Lib_v1" package="R1206" value="RES" x="39.6875" y="71.1835" rot="R90"/>
+<element name="U$1" library="Gas_Sensor_Lib_v1" package="SOT23" value="NMOS" x="38.608" y="76.327" smashed="yes" rot="R90">
+<attribute name="NAME" x="42.1005" y="75.057" size="1.27" layer="25" rot="R90"/>
+<attribute name="VALUE" x="43.8055" y="74.322" size="1.27" layer="27" rot="R90"/>
+</element>
+<element name="U$2" library="Gas_Sensor_Lib_v1" package="D-PAK_TO252AA" value="PMOS" x="29.718" y="60.198" smashed="yes" rot="R270">
+<attribute name="NAME" x="30.6945" y="52.933" size="1.27" layer="25" rot="R180"/>
+<attribute name="VALUE" x="28.0195" y="55.268" size="1.27" layer="27" rot="R180"/>
+</element>
+<element name="U$3" library="Gas_Sensor_Lib_v1" package="DIDOE_1206" value="DIODE_1206" x="11.43" y="58.4835" smashed="yes">
+<attribute name="NAME" x="10.16" y="59.7535" size="1.27" layer="25"/>
+<attribute name="VALUE" x="10.16" y="61.6585" size="1.27" layer="27"/>
+</element>
+<element name="U$4" library="Gas_Sensor_Lib_v1" package="R1206" value="10K" x="32.258" y="76.454" smashed="yes" rot="R180">
+<attribute name="NAME" x="33.528" y="74.549" size="1.27" layer="25" rot="R180"/>
+<attribute name="VALUE" x="33.528" y="78.994" size="1.27" layer="27" rot="R180"/>
+</element>
+<element name="U$5" library="Gas_Sensor_Lib_v1" package="R1206" value="100K" x="26.162" y="76.454" smashed="yes" rot="R180">
+<attribute name="NAME" x="27.432" y="74.549" size="1.27" layer="25" rot="R180"/>
+<attribute name="VALUE" x="27.432" y="72.644" size="1.27" layer="27" rot="R180"/>
+</element>
+<element name="U$6" library="Gas_Sensor_Lib_v1" package="R1206" value="1K" x="42.6085" y="61.214" smashed="yes" rot="R90">
+<attribute name="NAME" x="41.021" y="60.579" size="1.27" layer="25" rot="R90"/>
+<attribute name="VALUE" x="43.561" y="65.4685" size="1.27" layer="27" rot="R180"/>
+</element>
+<element name="U$7" library="Gas_Sensor_Lib_v1" package="R1206" value="100K" x="39.6875" y="71.1835" smashed="yes" rot="R90">
+<attribute name="NAME" x="42.8625" y="69.9135" size="1.27" layer="25" rot="R90"/>
+<attribute name="VALUE" x="38.1" y="68.6435" size="1.27" layer="27" rot="R90"/>
+</element>
 <element name="U$8" library="Gas_Sensor_Lib_v1" package="PC_1935161" value="POWER_CONN" x="5.08" y="46.101" rot="R270"/>
 <element name="U$9" library="Gas_Sensor_Lib_v1" package="ESP" value="ESP8266" x="29.591" y="24.892"/>
-<element name="U$10" library="Gas_Sensor_Lib_v1" package="R1206" value="RES" x="20.32" y="69.85"/>
-<element name="U$11" library="Gas_Sensor_Lib_v1" package="R1206" value="RES" x="42.545" y="51.6255" rot="R270"/>
+<element name="U$10" library="Gas_Sensor_Lib_v1" package="R1206" value="100" x="20.32" y="69.85" smashed="yes">
+<attribute name="NAME" x="19.05" y="71.755" size="1.27" layer="25"/>
+<attribute name="VALUE" x="19.05" y="73.66" size="1.27" layer="27"/>
+</element>
+<element name="U$11" library="Gas_Sensor_Lib_v1" package="R1206" value="10K" x="40.64" y="51.6255" smashed="yes" rot="R270">
+<attribute name="NAME" x="42.545" y="53.5305" size="1.27" layer="25" rot="R270"/>
+<attribute name="VALUE" x="40.3225" y="54.483" size="1.27" layer="27"/>
+</element>
 <element name="U$12" library="Gas_Sensor_Lib_v1" package="BUTTON" value="BUTTON" x="8.89" y="71.5645" smashed="yes" rot="R90"/>
-<element name="U$13" library="Gas_Sensor_Lib_v1" package="LED_1206" value="LED_1206" x="3.81" y="25.4" smashed="yes" rot="R90">
-<attribute name="NAME" x="2.54" y="24.13" size="1.27" layer="25" rot="R90"/>
-</element>
-<element name="U$14" library="Gas_Sensor_Lib_v1" package="C1206" value="CAP" x="14.097" y="16.383" rot="R90"/>
-<element name="U$15" library="Gas_Sensor_Lib_v1" package="R1206" value="RES" x="9.0805" y="22.86" rot="R270"/>
-<element name="U$16" library="Gas_Sensor_Lib_v1" package="R1206" value="RES" x="3.81" y="34.29" rot="R270"/>
+<element name="U$13" library="Gas_Sensor_Lib_v1" package="LED_1206" value="LED_12V" x="3.81" y="25.4" smashed="yes" rot="R90">
+<attribute name="NAME" x="6.0325" y="30.1625" size="1.27" layer="25" rot="R180"/>
+<attribute name="VALUE" x="1.905" y="22.225" size="1.27" layer="27" rot="R90"/>
+</element>
+<element name="U$14" library="Gas_Sensor_Lib_v1" package="C1206" value="470uF" x="14.097" y="16.383" smashed="yes" rot="R90">
+<attribute name="NAME" x="16.002" y="13.7795" size="1.27" layer="25" rot="R180"/>
+<attribute name="VALUE" x="16.637" y="12.192" size="1.27" layer="27" rot="R180"/>
+</element>
+<element name="U$15" library="Gas_Sensor_Lib_v1" package="R1206" value="330" x="9.0805" y="22.86" smashed="yes" rot="R270">
+<attribute name="NAME" x="10.9855" y="24.13" size="1.27" layer="25" rot="R270"/>
+<attribute name="VALUE" x="12.8905" y="24.13" size="1.27" layer="27" rot="R270"/>
+</element>
+<element name="U$16" library="Gas_Sensor_Lib_v1" package="R1206" value="1K" x="3.81" y="34.29" rot="R270"/>
 <element name="U$17" library="Gas_Sensor_Lib_v1" package="DIDOE_1206" value="DIODE_1206" x="3.81" y="16.51" smashed="yes" rot="R90">
 <attribute name="NAME" x="2.54" y="15.24" size="1.27" layer="25" rot="R90"/>
 </element>
-<element name="U$18" library="Gas_Sensor_Lib_v1" package="PC_1935161" value="POWER_CONN" x="8.255" y="5.0165"/>
-<element name="U$20" library="Gas_Sensor_Lib_v1" package="Z_1005" value="DIODE_Z_1005" x="9.144" y="16.129" rot="R270"/>
+<element name="U$18" library="Gas_Sensor_Lib_v1" package="PC_1935161" value="5V-12V" x="8.255" y="5.0165" smashed="yes">
+<attribute name="NAME" x="14.6135" y="3.255" size="1.016" layer="25" rot="R90"/>
+</element>
+<element name="U$20" library="Gas_Sensor_Lib_v1" package="Z_1005" value="15V_Z" x="9.144" y="16.129" smashed="yes" rot="R270">
+<attribute name="NAME" x="7.1835" y="11.114" size="1.27" layer="25"/>
+<attribute name="VALUE" x="6.5485" y="12.519" size="1.27" layer="27"/>
+</element>
 </elements>
 <signals>
@@
 <polygon width="0.4064" layer="1">
 <vertex x="0" y="80.01"/>
-<vertex x="48.006" y="80.01"/>
-<vertex x="48.006" y="0"/>
+<vertex x="44.196" y="80.01"/>
+<vertex x="44.196" y="0"/>
 <vertex x="0" y="0"/>
 </polygon>
 <polygon width="0.4064" layer="16">
 <vertex x="0" y="80.01"/>
-<vertex x="47.9425" y="80.0735"/>
-<vertex x="47.9425" y="0.0635"/>
+<vertex x="44.1325" y="80.0735"/>
+<vertex x="44.1325" y="0.0635"/>
 <vertex x="0" y="0"/>
 </polygon>
@@
 <contactref element="U$9" pad="GPIO4"/>
 <contactref element="U$6" pad="1"/>
-<wire x1="42.6085" y1="59.792" x2="42.6085" y2="57.3405" width="1.4224" layer="1"/>
-<wire x1="42.6085" y1="57.3405" x2="45.466" y2="54.483" width="1.4224" layer="1"/>
-<wire x1="43.74125625" y1="37.5111" x2="42.5276" y2="37.5111" width="1.4224" layer="1"/>
-<wire x1="42.5276" y1="37.5111" x2="41.021" y2="37.592" width="1.4224" layer="1"/>
-<wire x1="45.466" y1="54.483" x2="45.466" y2="40.82334375" width="1.4224" layer="1"/>
-<wire x1="45.466" y1="40.82334375" x2="43.74125625" y2="37.5111" width="1.4224" layer="1"/>
+<wire x1="42.6085" y1="57.3405" x2="42.6085" y2="59.792" width="1.4224" layer="1"/>
+<wire x1="41.021" y1="37.592" x2="43.02125" y2="37.62375" width="1.4224" layer="1"/>
+<wire x1="43.02125" y1="37.62375" x2="43.02125" y2="56.99125" width="1.4224" layer="1"/>
+<wire x1="43.02125" y1="56.99125" x2="42.6085" y2="57.3405" width="1.4224" layer="1"/>
 </signal>
 <signal name="N$7">
@@
 <wire x1="19.2005" y1="69.0645" x2="38.0365" y2="50.2285" width="1.4224" layer="16"/>
 <via x="38.0365" y="50.2285" extent="1-16" drill="1" shape="square"/>
-<wire x1="38.0365" y1="50.2285" x2="42.52" y2="50.2285" width="1.4224" layer="1"/>
-<wire x1="42.545" y1="50.2035" x2="42.52" y2="50.2285" width="1.4224" layer="1"/>
 <wire x1="41.021" y1="32.512" x2="38.1" y2="32.512" width="1.4224" layer="1"/>
-<wire x1="38.1" y1="50.165" x2="38.0365" y2="50.2285" width="1.4224" layer="1"/>
+<wire x1="38.0365" y1="50.2285" x2="38.1" y2="50.165" width="1.4224" layer="1"/>
 <wire x1="38.1" y1="32.512" x2="38.1" y2="50.165" width="1.4224" layer="1"/>
+<wire x1="40.64" y1="50.2035" x2="38.0365" y2="50.2285" width="1.4224" layer="1"/>
 </signal>
 <signal name="N$9">

Commit message: Add files via upload
I added an output LED on the receiver side and put some silkscreen on the bottom with our first names. 
I also added "RESET" next to the button on the silkscreen for the rx.
Input capacitance decreased to 10uF. Too expensive to get 470uF.
Parts:
- added U$19: OUT_LED, Gas_Sensor_Lib_v1:LED_1206
- added U$21: 1K, Gas_Sensor_Lib_v1:R1206
- U$14: value 470uF -> 10uF
- moved U$14 8.75 mm to (7.33, 10.8), turned to 0 degrees
Connections:
- new net N$5: U$19.2, U$21.2
- net GND: now also U$21.1
- net N$6: now also U$19.1
Routing:
- net N$6: track 60.4 -> 65.0 mm
- net N$5: track 0.00 -> 3.03 mm
- net 12V_IN: track 22.3 -> 19.7 mm
Other:
- board text added: "Alec Arsalan Kam Noah"
- board text added: "RECEIVER - RX CAPSTONE SPRING 2017"
- board text added: "RESET"
Changed lines of the file:
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@@
 <setting verticaltext="up"/>
 </settings>
-<grid distance="0.0125" unitdist="inch" unit="inch" style="dots" multiple="1" display="yes" altdistance="0.025" altunitdist="inch" altunit="inch"/>
+<grid distance="0.00625" unitdist="inch" unit="inch" style="dots" multiple="1" display="yes" altdistance="0.025" altunitdist="inch" altunit="inch"/>
 <layers>
 <layer number="1" name="Top" color="4" fill="1" visible="yes" active="yes"/>
@@
 <wire x1="0" y1="80.01" x2="0" y2="0" width="0" layer="20"/>
 <text x="0.6985" y="12.573" size="1.778" layer="21" rot="R270">12V_VIN</text>
-<text x="3.7465" y="51.8795" size="1.778" layer="21">LOAD</text>
+<text x="9.49325" y="47.21225" size="1.778" layer="21" rot="R270">LOAD</text>
+<text x="0.15875" y="77.94625" size="1.778" layer="21">RESET</text>
+<text x="38.4175" y="29.21" size="1.778" layer="22" rot="MR270">RECEIVER - RX
+CAPSTONE SPRING 2017</text>
+<text x="32.54375" y="9.68375" size="1.778" layer="22" rot="MR270">Alec
+Arsalan
+Kam
+Noah</text>
 </plain>
 <attributes>
@@
 <attribute name="VALUE" x="1.905" y="22.225" size="1.27" layer="27" rot="R90"/>
 </element>
-<element name="U$14" library="Gas_Sensor_Lib_v1" package="C1206" value="470uF" x="14.097" y="16.383" smashed="yes" rot="R90">
-<attribute name="NAME" x="16.002" y="13.7795" size="1.27" layer="25" rot="R180"/>
-<attribute name="VALUE" x="16.637" y="12.192" size="1.27" layer="27" rot="R180"/>
+<element name="U$14" library="Gas_Sensor_Lib_v1" package="C1206" value="10uF" x="7.33425" y="10.82675" smashed="yes">
+<attribute name="NAME" x="11.08075" y="9.398" size="1.27" layer="25" rot="R90"/>
+<attribute name="VALUE" x="12.66825" y="9.23925" size="1.27" layer="27" rot="R90"/>
 </element>
 <element name="U$15" library="Gas_Sensor_Lib_v1" package="R1206" value="330" x="9.0805" y="22.86" smashed="yes" rot="R270">
@@
 </element>
 <element name="U$20" library="Gas_Sensor_Lib_v1" package="Z_1005" value="15V_Z" x="9.144" y="16.129" smashed="yes" rot="R270">
-<attribute name="NAME" x="7.1835" y="11.114" size="1.27" layer="25"/>
-<attribute name="VALUE" x="6.5485" y="12.519" size="1.27" layer="27"/>
+<attribute name="NAME" x="13.49225" y="14.32725" size="1.27" layer="25" rot="R90"/>
+<attribute name="VALUE" x="11.9285" y="14.32725" size="1.27" layer="27" rot="R90"/>
+</element>
+<element name="U$19" library="Gas_Sensor_Lib_v1" package="LED_1206" value="OUT_LED" x="6.985" y="55.245" smashed="yes" rot="R180">
+<attribute name="NAME" x="8.5725" y="60.325" size="1.27" layer="25" rot="R180"/>
+<attribute name="VALUE" x="10.95375" y="53.18125" size="1.27" layer="27" rot="R180"/>
+</element>
+<element name="U$21" library="Gas_Sensor_Lib_v1" package="R1206" value="1K" x="2.54" y="56.67375" smashed="yes" rot="R270">
+<attribute name="NAME" x="1.27" y="61.11875" size="1.27" layer="25"/>
+<attribute name="VALUE" x="1.27" y="59.53125" size="1.27" layer="27"/>
 </element>
 </elements>
@@
 </polygon>
 <contactref element="U$8" pad="2"/>
+<contactref element="U$21" pad="1"/>
 </signal>
 <signal name="N$3">
@@
 <contactref element="U$2" pad="4"/>
 <contactref element="U$3" pad="2"/>
-<wire x1="12.852" y1="51.664" x2="12.852" y2="58.4835" width="1.4224" layer="1"/>
+<wire x1="12.852" y1="55.40375" x2="12.852" y2="51.664" width="1.4224" layer="1"/>
 <via x="14.6685" y="49.8475" extent="1-16" drill="1" shape="square"/>
+<wire x1="12.852" y1="55.40375" x2="12.852" y2="58.4835" width="1.4224" layer="1"/>
 <wire x1="14.6685" y1="49.8475" x2="17.272" y2="47.244" width="1.4224" layer="16"/>
 <wire x1="17.272" y1="47.244" x2="33.4645" y2="47.244" width="1.4224" layer="16"/>
@@
 <contactref element="U$8" pad="1"/>
 <wire x1="12.852" y1="48.601" x2="5.08" y2="48.601" width="1.4224" layer="1"/>
-<wire x1="12.852" y1="58.4835" x2="12.852" y2="48.601" width="1.4224" layer="1"/>
+<wire x1="12.852" y1="58.4835" x2="12.852" y2="55.40375" width="1.4224" layer="1"/>
+<contactref element="U$19" pad="1"/>
+<wire x1="12.852" y1="55.40375" x2="12.852" y2="48.601" width="1.4224" layer="1"/>
+<wire x1="8.407" y1="55.245" x2="12.852" y2="55.245" width="1.4224" layer="1"/>
+<wire x1="12.852" y1="55.245" x2="12.852" y2="55.40375" width="1.4224" layer="1"/>
 </signal>
 <signal name="N$2">
@@
 <contactref element="U$17" pad="1"/>
 <wire x1="5.755" y1="5.0165" x2="3.7465" y2="5.08" width="1.4224" layer="1"/>
-<wire x1="3.7465" y1="5.08" x2="3.81" y2="15.088" width="1.4224" layer="1"/>
+<wire x1="3.7837875" y1="10.9569375" x2="3.7465" y2="5.08" width="1.4224" layer="1"/>
+<wire x1="3.7837875" y1="10.9569375" x2="3.81" y2="15.088" width="1.4224" layer="1"/>
 <wire x1="3.81" y1="15.088" x2="9.144" y2="15.088" width="1.4224" layer="1"/>
 <wire x1="9.144" y1="15.088" x2="9.144" y2="15.129" width="1.4224" layer="1"/>
-<wire x1="9.144" y1="15.129" x2="14.097" y2="14.983" width="1.4224" layer="1"/>
+<wire x1="5.93425" y1="10.82675" x2="3.7837875" y2="10.82675" width="1.6764" layer="1"/>
+<wire x1="3.7837875" y1="10.82675" x2="3.7837875" y2="10.9569375" width="1.6764" layer="1"/>
 </signal>
 <signal name="12V">
@@
 <wire x1="9.0805" y1="21.438" x2="9.144" y2="17.129" width="1.4224" layer="1"/>
 </signal>
+<signal name="N$5">
+<contactref element="U$19" pad="2"/>
+<contactref element="U$21" pad="2"/>
+<wire x1="5.563" y1="55.245" x2="2.54" y2="55.245" width="1.4224" layer="1"/>
+<wire x1="2.54" y1="55.245" x2="2.54" y2="55.25175" width="1.4224" layer="1"/>
+</signal>
 </signals>
 </board>
 </drawing>
+<compatibility>
+<note version="6.3" minversion="6.2.2" severity="warning">
+Since Version 6.2.2 text objects can contain more than one line,
+which will not be processed correctly with this version.
+</note>
+</compatibility>
 </eagle>

Commit message: Fixed major error on tx board. Cap overlapped connector
Parts:
- moved U$14 0.81 mm to (7.18, 11.6)
Routing:
- net 12V_IN: track 19.7 -> 17.4 mm
Changed lines of the file:
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@@
 <text x="9.49325" y="47.21225" size="1.778" layer="21" rot="R270">LOAD</text>
 <text x="0.15875" y="77.94625" size="1.778" layer="21">RESET</text>
-<text x="38.4175" y="29.21" size="1.778" layer="22" rot="MR270">RECEIVER - RX
+<text x="38.57625" y="31.90875" size="1.778" layer="22" rot="MR270">RECEIVER - RX
 CAPSTONE SPRING 2017</text>
-<text x="32.54375" y="9.68375" size="1.778" layer="22" rot="MR270">Alec
+<text x="32.54375" y="12.54125" size="1.778" layer="22" rot="MR270">Alec
 Arsalan
 Kam
@@
 <attribute name="VALUE" x="1.905" y="22.225" size="1.27" layer="27" rot="R90"/>
 </element>
-<element name="U$14" library="Gas_Sensor_Lib_v1" package="C1206" value="10uF" x="7.33425" y="10.82675" smashed="yes">
-<attribute name="NAME" x="11.08075" y="9.398" size="1.27" layer="25" rot="R90"/>
-<attribute name="VALUE" x="12.66825" y="9.23925" size="1.27" layer="27" rot="R90"/>
+<element name="U$14" library="Gas_Sensor_Lib_v1" package="C1206" value="10uF" x="7.1755" y="11.6205" smashed="yes">
+<attribute name="NAME" x="10.922" y="9.7155" size="1.27" layer="25" rot="R90"/>
+<attribute name="VALUE" x="12.5095" y="9.7155" size="1.27" layer="27" rot="R90"/>
 </element>
 <element name="U$15" library="Gas_Sensor_Lib_v1" package="R1206" value="330" x="9.0805" y="22.86" smashed="yes" rot="R270">
@@
 <contactref element="U$20" pad="2"/>
 <contactref element="U$17" pad="1"/>
-<wire x1="5.755" y1="5.0165" x2="3.7465" y2="5.08" width="1.4224" layer="1"/>
-<wire x1="3.7837875" y1="10.9569375" x2="3.7465" y2="5.08" width="1.4224" layer="1"/>
-<wire x1="3.7837875" y1="10.9569375" x2="3.81" y2="15.088" width="1.4224" layer="1"/>
 <wire x1="3.81" y1="15.088" x2="9.144" y2="15.088" width="1.4224" layer="1"/>
 <wire x1="9.144" y1="15.088" x2="9.144" y2="15.129" width="1.4224" layer="1"/>
-<wire x1="5.93425" y1="10.82675" x2="3.7837875" y2="10.82675" width="1.6764" layer="1"/>
-<wire x1="3.7837875" y1="10.82675" x2="3.7837875" y2="10.9569375" width="1.6764" layer="1"/>
+<wire x1="5.755" y1="5.0165" x2="5.7755" y2="5.0165" width="1.6764" layer="1"/>
+<wire x1="5.7755" y1="5.0165" x2="5.7755" y2="11.6205" width="1.6764" layer="1"/>
+<wire x1="5.7755" y1="11.6205" x2="5.7755" y2="15.088" width="1.6764" layer="1"/>
+<wire x1="5.7755" y1="15.088" x2="3.81" y2="15.088" width="1.6764" layer="1"/>
 </signal>
 <signal name="12V">
