File: Schematic and Layout/Tx.sch (EAGLE design)
At the start: 31 parts

Commit message: Add files via upload
Parts:
- U$1: value LED_1206 -> LED_12V
- U$10, U$9: value CAP_POL -> 10uF
- U$11: value LED_1206 -> LED_5V
- U$12, U$15, U$21, U$23, U$27, U$4: value RES -> 1K
- U$16: value RES -> 5.1
- U$17, U$18: value CAP -> 100nF
- U$19: value LED_1206 -> LED_GAS
- U$2: value CAP -> 470u
- U$20: value DIODE_Z_1005 -> 15V_Z
- U$22: value RES -> 100K
- U$24: value CAP -> 1uF
- U$25, U$26: value RES -> ?
- U$3: value RES -> 330
- U$5: value DIODE_1206 -> DIODE
Changed lines of the file:
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@@
 </classes>
 <parts>
-<part name="U$1" library="Gas_Sensor_Lib_v1" deviceset="LED_1206" device=""/>
+<part name="U$1" library="Gas_Sensor_Lib_v1" deviceset="LED_1206" device="" value="LED_12V"/>
 <part name="GND3" library="supply1" deviceset="GND" device=""/>
-<part name="U$2" library="Gas_Sensor_Lib_v1" deviceset="CAP" device=""/>
-<part name="U$3" library="Gas_Sensor_Lib_v1" deviceset="RES" device=""/>
-<part name="U$4" library="Gas_Sensor_Lib_v1" deviceset="RES" device=""/>
-<part name="U$5" library="Gas_Sensor_Lib_v1" deviceset="DIODE_1206" device=""/>
+<part name="U$2" library="Gas_Sensor_Lib_v1" deviceset="CAP" device="" value="470u"/>
+<part name="U$3" library="Gas_Sensor_Lib_v1" deviceset="RES" device="" value="330"/>
+<part name="U$4" library="Gas_Sensor_Lib_v1" deviceset="RES" device="" value="1K"/>
+<part name="U$5" library="Gas_Sensor_Lib_v1" deviceset="DIODE_1206" device="" value="DIODE"/>
 <part name="U$6" library="Gas_Sensor_Lib_v1" deviceset="POWER_CONN" device=""/>
 <part name="U$7" library="Gas_Sensor_Lib_v1" deviceset="LM393" device=""/>
 <part name="U$8" library="Gas_Sensor_Lib_v1" deviceset="5V_REG" device=""/>
-<part name="U$9" library="Gas_Sensor_Lib_v1" deviceset="CAP_POL" device=""/>
-<part name="U$10" library="Gas_Sensor_Lib_v1" deviceset="CAP_POL" device=""/>
+<part name="U$9" library="Gas_Sensor_Lib_v1" deviceset="CAP_POL" device="" value="10uF"/>
+<part name="U$10" library="Gas_Sensor_Lib_v1" deviceset="CAP_POL" device="" value="10uF"/>
 <part name="GND1" library="supply1" deviceset="GND" device=""/>
 <part name="GND2" library="supply1" deviceset="GND" device=""/>
-<part name="U$11" library="Gas_Sensor_Lib_v1" deviceset="LED_1206" device=""/>
-<part name="U$12" library="Gas_Sensor_Lib_v1" deviceset="RES" device=""/>
+<part name="U$11" library="Gas_Sensor_Lib_v1" deviceset="LED_1206" device="" value="LED_5V"/>
+<part name="U$12" library="Gas_Sensor_Lib_v1" deviceset="RES" device="" value="1K"/>
 <part name="U$13" library="Gas_Sensor_Lib_v1" deviceset="MQ" device=""/>
 <part name="U$14" library="Gas_Sensor_Lib_v1" deviceset="PNP" device=""/>
-<part name="U$15" library="Gas_Sensor_Lib_v1" deviceset="RES" device=""/>
+<part name="U$15" library="Gas_Sensor_Lib_v1" deviceset="RES" device="" value="1K"/>
 <part name="GND4" library="supply1" deviceset="GND" device=""/>
-<part name="U$16" library="Gas_Sensor_Lib_v1" deviceset="RES" device=""/>
+<part name="U$16" library="Gas_Sensor_Lib_v1" deviceset="RES" device="" value="5.1"/>
 <part name="GND5" library="supply1" deviceset="GND" device=""/>
 <part name="GND6" library="supply1" deviceset="GND" device=""/>
-<part name="U$17" library="Gas_Sensor_Lib_v1" deviceset="CAP" device=""/>
+<part name="U$17" library="Gas_Sensor_Lib_v1" deviceset="CAP" device="" value="100nF"/>
 <part name="GND7" library="supply1" deviceset="GND" device=""/>
-<part name="U$18" library="Gas_Sensor_Lib_v1" deviceset="CAP" device=""/>
-<part name="U$19" library="Gas_Sensor_Lib_v1" deviceset="LED_1206" device=""/>
-<part name="U$20" library="Gas_Sensor_Lib_v1" deviceset="DIODE_Z_1005" device=""/>
-<part name="U$21" library="Gas_Sensor_Lib_v1" deviceset="RES" device=""/>
+<part name="U$18" library="Gas_Sensor_Lib_v1" deviceset="CAP" device="" value="100nF"/>
+<part name="U$19" library="Gas_Sensor_Lib_v1" deviceset="LED_1206" device="" value="LED_GAS"/>
+<part name="U$20" library="Gas_Sensor_Lib_v1" deviceset="DIODE_Z_1005" device="" value="15V_Z"/>
+<part name="U$21" library="Gas_Sensor_Lib_v1" deviceset="RES" device="" value="1K"/>
 <part name="GND8" library="supply1" deviceset="GND" device=""/>
-<part name="U$22" library="Gas_Sensor_Lib_v1" deviceset="RES" device=""/>
-<part name="U$23" library="Gas_Sensor_Lib_v1" deviceset="RES" device=""/>
-<part name="U$24" library="Gas_Sensor_Lib_v1" deviceset="CAP" device=""/>
-<part name="U$25" library="Gas_Sensor_Lib_v1" deviceset="RES" device=""/>
-<part name="U$26" library="Gas_Sensor_Lib_v1" deviceset="RES" device=""/>
-<part name="U$27" library="Gas_Sensor_Lib_v1" deviceset="RES" device=""/>
+<part name="U$22" library="Gas_Sensor_Lib_v1" deviceset="RES" device="" value="100K"/>
+<part name="U$23" library="Gas_Sensor_Lib_v1" deviceset="RES" device="" value="1K"/>
+<part name="U$24" library="Gas_Sensor_Lib_v1" deviceset="CAP" device="" value="1uF"/>
+<part name="U$25" library="Gas_Sensor_Lib_v1" deviceset="RES" device="" value="?"/>
+<part name="U$26" library="Gas_Sensor_Lib_v1" deviceset="RES" device="" value="?"/>
+<part name="U$27" library="Gas_Sensor_Lib_v1" deviceset="RES" device="" value="1K"/>
 <part name="U$28" library="Gas_Sensor_Lib_v1" deviceset="DIODE_1206" device=""/>
 <part name="GND9" library="supply1" deviceset="GND" device=""/>

Commit message: Add files via upload
I added an output LED on the receiver side and put some silkscreen on the bottom with our first names. 
I also added "RESET" next to the button on the silkscreen for the rx.
Input capacitance decreased to 10uF. Too expensive to get 470uF.
Parts:
- U$2: value 470u -> 10uF
Changed lines of the file:
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@@
 <part name="U$1" library="Gas_Sensor_Lib_v1" deviceset="LED_1206" device="" value="LED_12V"/>
 <part name="GND3" library="supply1" deviceset="GND" device=""/>
-<part name="U$2" library="Gas_Sensor_Lib_v1" deviceset="CAP" device="" value="470u"/>
+<part name="U$2" library="Gas_Sensor_Lib_v1" deviceset="CAP" device="" value="10uF"/>
 <part name="U$3" library="Gas_Sensor_Lib_v1" deviceset="RES" device="" value="330"/>
 <part name="U$4" library="Gas_Sensor_Lib_v1" deviceset="RES" device="" value="1K"/>

Commit message: Major error fixed, was missing 5V on PNP
Connections:
- removed net N$10: U$14.E, U$22.1, U$24.1
- net 5V: now also U$14.E, U$22.1, U$24.1
Changed lines of the file:
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@@
 <label x="121.92" y="30.48" size="1.778" layer="95"/>
+</segment>
+<segment>
+<pinref part="U$22" gate="G$1" pin="1"/>
+<wire x1="269.24" y1="129.54" x2="269.24" y2="132.08" width="0.1524" layer="91"/>
+<wire x1="269.24" y1="132.08" x2="281.94" y2="132.08" width="0.1524" layer="91"/>
+<pinref part="U$14" gate="G$1" pin="E"/>
+<wire x1="281.94" y1="132.08" x2="281.94" y2="116.84" width="0.1524" layer="91"/>
+<pinref part="U$24" gate="G$1" pin="1"/>
+<wire x1="281.94" y1="116.84" x2="289.56" y2="116.84" width="0.1524" layer="91"/>
+<wire x1="289.56" y1="116.84" x2="289.56" y2="114.3" width="0.1524" layer="91"/>
+<junction x="281.94" y="116.84"/>
+<label x="271.78" y="132.08" size="1.778" layer="95"/>
 </segment>
 </net>
@@
 </segment>
 </net>
-<net name="N$10" class="0">
-<segment>
-<pinref part="U$22" gate="G$1" pin="1"/>
-<wire x1="269.24" y1="129.54" x2="269.24" y2="132.08" width="0.1524" layer="91"/>
-<wire x1="269.24" y1="132.08" x2="281.94" y2="132.08" width="0.1524" layer="91"/>
-<pinref part="U$14" gate="G$1" pin="E"/>
-<wire x1="281.94" y1="132.08" x2="281.94" y2="116.84" width="0.1524" layer="91"/>
-<pinref part="U$24" gate="G$1" pin="1"/>
-<wire x1="281.94" y1="116.84" x2="289.56" y2="116.84" width="0.1524" layer="91"/>
-<wire x1="289.56" y1="116.84" x2="289.56" y2="114.3" width="0.1524" layer="91"/>
-<junction x="281.94" y="116.84"/>
-</segment>
-</net>

Commit message: ESPs now run off of 5 V
Parts:
- added U$32: SPDT, Gas_Sensor_Lib_v1:SPDT
Connections:
- new net ESP_VIN: U$29.VIN, U$32.A
- net 12V: no longer U$29.VIN
- net 5V: now also U$32.INPUT
Changed lines of the file:
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@@
 <part name="GND11" library="supply1" deviceset="GND" device=""/>
 <part name="U$31" library="Gas_Sensor_Lib_v1" deviceset="HEAT_SINK" device=""/>
+<part name="U$32" library="Gas_Sensor_Lib_v1" deviceset="SPDT" device=""/>
 </parts>
 <sheets>
@@
 <instance part="GND11" gate="1" x="187.96" y="22.86"/>
 <instance part="U$31" gate="G$1" x="66.04" y="119.38"/>
+<instance part="U$32" gate="G$1" x="332.74" y="109.22"/>
 </instances>
 <busses>
@@
 <junction x="111.76" y="147.32"/>
 <label x="83.82" y="182.88" size="1.778" layer="95"/>
-</segment>
-<segment>
-<pinref part="U$29" gate="G$1" pin="VIN"/>
-<wire x1="320.04" y1="88.9" x2="314.96" y2="88.9" width="0.1524" layer="91"/>
-<wire x1="314.96" y1="88.9" x2="314.96" y2="99.06" width="0.1524" layer="91"/>
-<label x="314.96" y="96.52" size="1.778" layer="95"/>
 </segment>
 </net>
@@
 <label x="271.78" y="132.08" size="1.778" layer="95"/>
 </segment>
+<segment>
+<label x="350.52" y="96.52" size="1.778" layer="95"/>
+<pinref part="U$32" gate="G$1" pin="INPUT"/>
+<wire x1="332.74" y1="101.6" x2="332.74" y2="96.52" width="0.1524" layer="91"/>
+<wire x1="332.74" y1="96.52" x2="355.6" y2="96.52" width="0.1524" layer="91"/>
+</segment>
 </net>
 <net name="N$3" class="0">
@@
 </segment>
 </net>
+<net name="ESP_VIN" class="0">
+<segment>
+<pinref part="U$29" gate="G$1" pin="VIN"/>
+<wire x1="320.04" y1="88.9" x2="314.96" y2="88.9" width="0.1524" layer="91"/>
+<label x="314.96" y="96.52" size="1.778" layer="95"/>
+<pinref part="U$32" gate="G$1" pin="A"/>
+<wire x1="314.96" y1="88.9" x2="314.96" y2="101.6" width="0.1524" layer="91"/>
+<wire x1="314.96" y1="101.6" x2="325.12" y2="101.6" width="0.1524" layer="91"/>
+</segment>
+</net>

Commit message: Definitively added zener diodes
Parts:
- removed U$26: ?, Gas_Sensor_Lib_v1:RES
- U$25: value ? -> 1K
- U$28: value DIODE_1206 -> DIODE_Z_3.3V; device Gas_Sensor_Lib_v1:DIODE_1206 -> Gas_Sensor_Lib_v1:DIODE_Z_3.3V
Connections:
- removed net N$12: U$26.1, U$28.HI
- net GND: now also U$28.HI; no longer U$28.LO
- net N$13: now also U$28.LO; no longer U$26.2
Changed lines of the file:
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@@
 <part name="U$23" library="Gas_Sensor_Lib_v1" deviceset="RES" device="" value="1K"/>
 <part name="U$24" library="Gas_Sensor_Lib_v1" deviceset="CAP" device="" value="1uF"/>
-<part name="U$25" library="Gas_Sensor_Lib_v1" deviceset="RES" device="" value="?"/>
-<part name="U$26" library="Gas_Sensor_Lib_v1" deviceset="RES" device="" value="?"/>
+<part name="U$25" library="Gas_Sensor_Lib_v1" deviceset="RES" device="" value="1K"/>
 <part name="U$27" library="Gas_Sensor_Lib_v1" deviceset="RES" device="" value="1K"/>
-<part name="U$28" library="Gas_Sensor_Lib_v1" deviceset="DIODE_1206" device=""/>
 <part name="GND9" library="supply1" deviceset="GND" device=""/>
 <part name="U$29" library="Gas_Sensor_Lib_v1" deviceset="ESP8266" device=""/>
@@
 <part name="U$31" library="Gas_Sensor_Lib_v1" deviceset="HEAT_SINK" device=""/>
 <part name="U$32" library="Gas_Sensor_Lib_v1" deviceset="SPDT" device=""/>
+<part name="U$28" library="Gas_Sensor_Lib_v1" deviceset="DIODE_Z_3.3V" device=""/>
 </parts>
 <sheets>
@@
 <instance part="U$24" gate="G$1" x="289.56" y="111.76"/>
 <instance part="U$25" gate="G$1" x="281.94" y="93.98" rot="R90"/>
-<instance part="U$26" gate="G$1" x="281.94" y="73.66" rot="R90"/>
 <instance part="U$27" gate="G$1" x="297.18" y="83.82" rot="R180"/>
-<instance part="U$28" gate="G$1" x="281.94" y="58.42"/>
 <instance part="GND9" gate="1" x="281.94" y="45.72"/>
 <instance part="U$29" gate="G$1" x="327.66" y="68.58"/>
@@
 <instance part="U$31" gate="G$1" x="66.04" y="119.38"/>
 <instance part="U$32" gate="G$1" x="332.74" y="109.22"/>
+<instance part="U$28" gate="G$1" x="281.94" y="58.42" rot="R180"/>
 </instances>
 <busses>
@@
 <pinref part="U$18" gate="G$1" pin="1"/>
 <wire x1="195.58" y1="96.52" x2="195.58" y2="101.6" width="0.1524" layer="91"/>
-</segment>
-<segment>
-<pinref part="GND9" gate="1" pin="GND"/>
-<pinref part="U$28" gate="G$1" pin="LO"/>
-<wire x1="281.94" y1="48.26" x2="281.94" y2="53.34" width="0.1524" layer="91"/>
 </segment>
 <segment>
@@
 <wire x1="180.34" y1="27.94" x2="187.96" y2="27.94" width="0.1524" layer="91"/>
 <junction x="187.96" y="27.94"/>
+</segment>
+<segment>
+<pinref part="GND9" gate="1" pin="GND"/>
+<pinref part="U$28" gate="G$1" pin="HI"/>
+<wire x1="281.94" y1="48.26" x2="281.94" y2="55.88" width="0.1524" layer="91"/>
 </segment>
 </net>
@@
 </segment>
 </net>
-<net name="N$12" class="0">
-<segment>
-<pinref part="U$28" gate="G$1" pin="HI"/>
-<pinref part="U$26" gate="G$1" pin="1"/>
-<wire x1="281.94" y1="60.96" x2="281.94" y2="68.58" width="0.1524" layer="91"/>
-</segment>
-</net>
 <net name="N$13" class="0">
 <segment>
-<pinref part="U$26" gate="G$1" pin="2"/>
 <pinref part="U$25" gate="G$1" pin="1"/>
-<wire x1="281.94" y1="78.74" x2="281.94" y2="83.82" width="0.1524" layer="91"/>
 <pinref part="U$27" gate="G$1" pin="2"/>
 <wire x1="281.94" y1="83.82" x2="281.94" y2="88.9" width="0.1524" layer="91"/>
 <wire x1="292.1" y1="83.82" x2="281.94" y2="83.82" width="0.1524" layer="91"/>
 <junction x="281.94" y="83.82"/>
-</segment>
-</net>
+<pinref part="U$28" gate="G$1" pin="LO"/>
+<wire x1="281.94" y1="83.82" x2="281.94" y2="63.5" width="0.1524" layer="91"/>
+</segment>
+</net>
